File: Power.sch (KiCad schematic (older format))
At the start: 13 parts, among them J3 Conn_01x02, Q1 SUD19P06-60, U1 LM2678

Commit message: Updated Library Refs
Parts:
- U1: symbol SMPS_Regulators:LM2678 -> _SMPS_Regulators:LM2678
Changed lines of the file:
@@
 $EndDescr
 $Comp
-L SMPS_Regulators:LM2678 U1
+L _SMPS_Regulators:LM2678 U1
 U 1 1 5FB73DAC
 P 4800 2500
